File: WiazkaLewaRekojesc.sch (EAGLE design)
At the start: 1 part, among them X6-B MSTBV_2,5/13-G

Commit message: rev.003 RC1
Connections:
- net KLAKSON(+12V) renamed KLAKSON(+12V/ST)
Changed lines of the file:
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@@
 <?xml version="1.0" encoding="utf-8"?>
 <!DOCTYPE eagle SYSTEM "eagle.dtd">
-<eagle version="7.7.0">
+<eagle version="8.6.0">
 <drawing>
 <settings>
 <setting alwaysvectorfont="no"/>
+<setting keepoldvectorfont="yes"/>
 <setting verticaltext="up"/>
 </settings>
@@
 </segment>
 </net>
-<net name="KLAKSON(+12V)" class="0">
+<net name="KLAKSON(+12V/ST)" class="0">
 <segment>
 <wire x1="124.46" y1="88.9" x2="124.46" y2="86.36" width="0.1524" layer="91"/>
