File: PlytaGlowna.sch (EAGLE design)
At the start: 17 parts, among them X10A- CZUJ_STOP_PRAWY, X11A- CZUJNIK_STOP_LEWY, X12A- SWIATL_PRZOD, X13A- SWIATL_TYL, X1B 5566-2, X2A- STACYJKA, X3A- VOLTOMIERZ, X4A- PRZERYWACZ, X5A- WL_SWIATLA_DZIENNE, X6A- REKOJESC_LEW, X7A- KLAKSON, X8A- ZAS USB/12V, X9A- SYGNALIZATOR

Commit message: druga wyprodukowana plytka
Parts:
- removed R1, R2, R3, R4: (no value), rcl:R-EU_R1206
- removed X5A-: WL_SWIATLA_DZIENNE, my_electronics_library:43045-0212
- added D1, D2: 1N4446, diode:1N4446
- added U$1: 43045-0412, my_electronics_library:43045-0412
- added U$2: BUZZER, my_electronics_library:43045-0212
Connections:
- removed net N$2: R2.2, X9A-G$2.S
- removed net N$3: R3.2, X9A-G$3.S
- removed net N$4: R4.2, X9A-G$5.S
- net +12V: no longer X6A-G$4.S
- net +12V/ST: now also U$1G$2.S, X6A-G$4.S, X9A-G$5.S; no longer R4.1, X5A-G$1.S
- net DZIENNE: now also U$1G$1.S; no longer X5A-G$2.S
- net KIER_LEWY: now also D1.A, X9A-G$1.S; no longer R1.1
- net KIER_PRAWY: now also D2.A, X9A-G$2.S; no longer R2.1
- net MASA: now also U$1G$3.S, U$2G$2.S
- net MIJANIA: now also X9A-G$3.S; no longer R3.1
- net N$1: now also D1.C, D2.C, U$2G$1.S; no longer R1.2, X9A-G$1.S
Other:
- moved on the sheet: X1B-1, X1B-2, X2A-G$1, X2A-G$2, X3A-G$1, X3A-G$2, X4A-G$1, X4A-G$2, X4A-G$3, X4A-G$4

Commit message: czesc zmian do wersji 3
Parts:
- removed U$2: BUZZER, my_electronics_library:43045-0212
- removed X2A-: STACYJKA, my_electronics_library:43045-0212
- removed X3A-: VOLTOMIERZ, my_electronics_library:43045-0212
- removed X4A-: PRZERYWACZ, my_electronics_library:43045-0412
- added J1: PRZERYWACZ, con-molex:22-27-2031-03
- added J2: STACYJKA, con-molex:22-27-2021-02
- added J3: VOLTOMIERZ, con-molex:22-27-2021-02
- added J4: BUZZER, con-molex:22-27-2021-02
Connections:
- net +12V: now also J2-1.S; no longer X2A-G$1.S
- net +12V/ST: now also J1-1.S, J2-2.S, J3-1.S; no longer X2A-G$2.S, X3A-G$1.S, X4A-G$1.S
- net KIER_WSPOLNY: now also J1-3.S; no longer X4A-G$3.S
- net MASA: now also J1-2.S, J3-2.S, J4-1.S; no longer U$2G$2.S, X3A-G$2.S, X4A-G$2.S
- net N$1: now also J4-2.S; no longer U$2G$1.S
Changed lines of the file:
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@@
 <?xml version="1.0" encoding="utf-8"?>
 <!DOCTYPE eagle SYSTEM "eagle.dtd">
-<eagle version="7.7.0">
+<eagle version="8.6.0">
 <drawing>
 <settings>
 <setting alwaysvectorfont="no"/>
+<setting keepoldvectorfont="yes"/>
 <setting verticaltext="up"/>
 </settings>
@@
 <parts>
 <part name="X1B" library="con-molex" deviceset="5566-2" device=""/>
-<part name="X2A-" library="my_electronics_library" deviceset="43045-0212" device="" value="STACYJKA"/>
-<part name="X3A-" library="my_electronics_library" deviceset="43045-0212" device="" value="VOLTOMIERZ"/>
 <part name="X7A-" library="my_electronics_library" deviceset="43045-0212" device="" value="KLAKSON"/>
 <part name="X8A-" library="my_electronics_library" deviceset="43045-0212" device="" value="ZAS USB/12V"/>
 <part name="X10A-" library="my_electronics_library" deviceset="43045-0212" device="" value="CZUJ_STOP_PRAWY"/>
 <part name="X11A-" library="my_electronics_library" deviceset="43045-0212" device="" value="CZUJNIK_STOP_LEWY"/>
-<part name="X4A-" library="my_electronics_library" deviceset="43045-0412" device="" value="PRZERYWACZ"/>
 <part name="X6A-" library="my_electronics_library" deviceset="43045-0812" device="" value="REKOJESC_LEW"/>
 <part name="X9A-" library="my_electronics_library" deviceset="43045-0612" device="" value="SYGNALIZATOR"/>
@@
 <part name="X13A-" library="my_electronics_library" deviceset="43045-0612" device="" value="SWIATL_TYL"/>
 <part name="U$1" library="my_electronics_library" deviceset="43045-0412" device=""/>
-<part name="U$2" library="my_electronics_library" deviceset="43045-0212" device="" value="BUZZER"/>
 <part name="D1" library="diode" deviceset="1N4446" device=""/>
 <part name="D2" library="diode" deviceset="1N4446" device=""/>
+<part name="J1" library="con-molex" library_urn="urn:adsk.eagle:library:165" deviceset="22-?-03" device="27-2031" value="PRZERYWACZ"/>
+<part name="J2" library="con-molex" library_urn="urn:adsk.eagle:library:165" deviceset="22-?-02" device="27-2021" value="STACYJKA"/>
+<part name="J3" library="con-molex" library_urn="urn:adsk.eagle:library:165" deviceset="22-?-02" device="27-2021" value="VOLTOMIERZ"/>
+<part name="J4" library="con-molex" library_urn="urn:adsk.eagle:library:165" deviceset="22-?-02" device="27-2021" value="BUZZER"/>
 </parts>
 <sheets>
@@
 <instance part="X1B" gate="-1" x="-35.56" y="93.98" rot="R180"/>
 <instance part="X1B" gate="-2" x="-35.56" y="88.9" rot="R180"/>
-<instance part="X2A-" gate="G$1" x="-10.16" y="127" rot="R90"/>
-<instance part="X2A-" gate="G$2" x="-5.08" y="127" rot="R90"/>
-<instance part="X3A-" gate="G$1" x="15.24" y="129.54" rot="R90"/>
-<instance part="X3A-" gate="G$2" x="20.32" y="129.54" rot="R90"/>
 <instance part="X7A-" gate="G$1" x="208.28" y="165.1" rot="R90"/>
 <instance part="X7A-" gate="G$2" x="200.66" y="165.1" rot="R90"/>
@@
 <instance part="X11A-" gate="G$1" x="340.36" y="160.02" rot="R90"/>
 <instance part="X11A-" gate="G$2" x="347.98" y="160.02" rot="R90"/>
-<instance part="X4A-" gate="G$1" x="33.02" y="124.46" rot="R90"/>
-<instance part="X4A-" gate="G$2" x="40.64" y="124.46" rot="R90"/>
-<instance part="X4A-" gate="G$3" x="48.26" y="124.46" rot="R90"/>
-<instance part="X4A-" gate="G$4" x="53.34" y="124.46" rot="R90"/>
 <instance part="X6A-" gate="G$1" x="144.78" y="213.36" rot="R90"/>
 <instance part="X6A-" gate="G$2" x="149.86" y="213.36" rot="R90"/>
@@
 <instance part="U$1" gate="G$3" x="96.52" y="172.72" rot="R90"/>
 <instance part="U$1" gate="G$4" x="101.6" y="172.72" rot="R90"/>
-<instance part="U$2" gate="G$1" x="378.46" y="160.02" rot="R90"/>
-<instance part="U$2" gate="G$2" x="383.54" y="160.02" rot="R90"/>
 <instance part="D1" gate="1" x="365.76" y="116.84" rot="R90"/>
 <instance part="D2" gate="1" x="370.84" y="116.84" rot="R90"/>
+<instance part="J1" gate="-1" x="33.02" y="124.46" rot="R90"/>
+<instance part="J1" gate="-2" x="40.64" y="124.46" rot="R90"/>
+<instance part="J1" gate="-3" x="48.26" y="124.46" rot="R90"/>
+<instance part="J2" gate="-1" x="-10.16" y="127" rot="R90"/>
+<instance part="J2" gate="-2" x="-5.08" y="127" rot="R90"/>
+<instance part="J3" gate="-1" x="15.24" y="129.54" rot="R90"/>
+<instance part="J3" gate="-2" x="20.32" y="129.54" rot="R90"/>
+<instance part="J4" gate="-1" x="383.54" y="160.02" rot="R90"/>
+<instance part="J4" gate="-2" x="378.46" y="160.02" rot="R90"/>
 </instances>
 <busses>
@@
 <wire x1="233.68" y1="121.92" x2="152.4" y2="121.92" width="0.1524" layer="91"/>
 <pinref part="X1B" gate="-1" pin="S"/>
-<pinref part="X2A-" gate="G$1" pin="S"/>
 <pinref part="X8A-" gate="G$2" pin="S"/>
 <wire x1="233.68" y1="167.64" x2="233.68" y2="121.92" width="0.1524" layer="91"/>
 <label x="-10.16" y="111.76" size="2.54" layer="95" rot="R90"/>
 <label x="233.68" y="147.32" size="2.54" layer="95" rot="R90"/>
+<pinref part="J2" gate="-1" pin="S"/>
 </segment>
 </net>
@@
 <junction x="40.64" y="76.2"/>
 <pinref part="X1B" gate="-2" pin="S"/>
-<pinref part="X4A-" gate="G$2" pin="S"/>
 <pinref part="X12A-" gate="G$6" pin="S"/>
 <wire x1="464.82" y1="152.4" x2="482.6" y2="152.4" width="0.1524" layer="91"/>
@@
 <wire x1="208.28" y1="162.56" x2="208.28" y2="76.2" width="0.1524" layer="91"/>
 <junction x="208.28" y="76.2"/>
-<pinref part="X3A-" gate="G$2" pin="S"/>
 <wire x1="20.32" y1="127" x2="20.32" y2="76.2" width="0.1524" layer="91"/>
 <junction x="20.32" y="76.2"/>
@@
 <wire x1="96.52" y1="170.18" x2="96.52" y2="76.2" width="0.1524" layer="91"/>
 <junction x="96.52" y="76.2"/>
-<pinref part="U$2" gate="G$2" pin="S"/>
 <wire x1="383.54" y1="157.48" x2="383.54" y2="58.42" width="0.1524" layer="91"/>
 <junction x="383.54" y="58.42"/>
+<pinref part="J1" gate="-2" pin="S"/>
+<pinref part="J3" gate="-2" pin="S"/>
+<pinref part="J4" gate="-1" pin="S"/>
 </segment>
 </net>
@@
 <wire x1="340.36" y1="91.44" x2="340.36" y2="157.48" width="0.1524" layer="91"/>
 <junction x="312.42" y="91.44"/>
-<pinref part="X2A-" gate="G$2" pin="S"/>
 <pinref part="X10A-" gate="G$1" pin="S"/>
 <pinref part="X11A-" gate="G$1" pin="S"/>
-<pinref part="X4A-" gate="G$1" pin="S"/>
 <pinref part="X6A-" gate="G$1" pin="S"/>
-<pinref part="X3A-" gate="G$1" pin="S"/>
 <wire x1="15.24" y1="127" x2="15.24" y2="91.44" width="0.1524" layer="91"/>
 <junction x="15.24" y="91.44"/>
@@
 <pinref part="U$1" gate="G$2" pin="S"/>
 <wire x1="91.44" y1="91.44" x2="91.44" y2="170.18" width="0.1524" layer="91"/>
+<pinref part="J1" gate="-1" pin="S"/>
+<pinref part="J2" gate="-2" pin="S"/>
+<pinref part="J3" gate="-1" pin="S"/>
 </segment>
 </net>
@@
 <wire x1="167.64" y1="193.04" x2="170.18" y2="193.04" width="0.1524" layer="91"/>
 <wire x1="170.18" y1="193.04" x2="170.18" y2="210.82" width="0.1524" layer="91"/>
-<pinref part="X4A-" gate="G$3" pin="S"/>
 <pinref part="X6A-" gate="G$6" pin="S"/>
 <label x="48.26" y="106.68" size="2.54" layer="95" rot="R90"/>
 <label x="167.64" y="182.88" size="2.54" layer="95" rot="R90"/>
+<pinref part="J1" gate="-3" pin="S"/>
 </segment>
 </net>
@@
 <pinref part="D2" gate="1" pin="C"/>
 <wire x1="365.76" y1="119.38" x2="370.84" y2="119.38" width="0.1524" layer="91"/>
-<pinref part="U$2" gate="G$1" pin="S"/>
 <wire x1="370.84" y1="119.38" x2="378.46" y2="119.38" width="0.1524" layer="91"/>
 <wire x1="378.46" y1="119.38" x2="378.46" y2="157.48" width="0.1524" layer="91"/>
 <junction x="370.84" y="119.38"/>
+<pinref part="J4" gate="-2" pin="S"/>
 </segment>
 </net>
@@
 </schematic>
 </drawing>
+<compatibility>
+<note version="8.2" severity="warning">
+Since Version 8.2, EAGLE supports online libraries. The ids
+of those online libraries will not be understood (or retained)
+with this version.
+</note>
+</compatibility>
 </eagle>

Commit message: temporary changes
Parts:
- removed U$1: 43045-0412, my_electronics_library:43045-0412
- removed X10A-: CZUJ_STOP_PRAWY, my_electronics_library:43045-0212
- removed X11A-: CZUJNIK_STOP_LEWY, my_electronics_library:43045-0212
- removed X12A-: SWIATL_PRZOD, my_electronics_library:43045-0612
- removed X13A-: SWIATL_TYL, my_electronics_library:43045-0612
- removed X7A-: KLAKSON, my_electronics_library:43045-0212
- removed X8A-: ZAS USB/12V, my_electronics_library:43045-0212
- removed X9A-: SYGNALIZATOR, my_electronics_library:43045-0612
- added J10: SWIATLA_TYL, con-molex:22-27-2061-06
- added J11: SWIATLA_PRZOD, con-molex:22-27-2061-06
- added J12: SYGNALIZATOR, con-molex:22-27-2061-06
- added J13: 22-27-2081-08, con-molex:22-27-2081-08
- added J5: KLAKSON, con-molex:22-27-2021-02
- added J6: CZUJNIK_STOP_LEWY, con-molex:22-27-2021-02
- added J7: CZUJNIK_STOP_PRAWY, con-molex:22-27-2021-02
- added J8: ZAS_USB/12V, con-molex:22-27-2021-02
- added J9: 22-27-2031-03, con-molex:22-27-2031-03
Connections:
- net +12V: now also J8-1.S; no longer X8A-G$2.S
- net +12V/ST: now also J12-3.S, J6-1.S, J7-1.S, J9-1.S; no longer U$1G$2.S, X10A-G$1.S, X11A-G$1.S, X9A-G$5.S
- net DZIENNE: now also J11-4.S, J9-2.S; no longer U$1G$1.S, X12A-G$2.S
- net KIER_LEWY: now also J10-1.S, J11-6.S, J12-1.S; no longer X12A-G$4.S, X13A-G$6.S, X9A-G$1.S
- net KIER_PRAWY: now also J10-3.S, J11-3.S, J12-2.S; no longer X12A-G$5.S, X13A-G$5.S, X9A-G$2.S
- net KLAKSON: now also J5-1.S; no longer X7A-G$2.S
- net MASA: now also J10-5.S, J10-6.S, J11-1.S, J11-2.S, J12-5.S, J5-2.S, J8-2.S, J9-3.S; no longer U$1G$3.S, X12A-G$6.S, X13A-G$4.S, X7A-G$1.S, X8A-G$1.S, X9A-G$6.S
- net MIJANIA: now also J10-2.S, J11-5.S, J12-6.S; no longer X12A-G$1.S, X13A-G$3.S, X9A-G$3.S
- net STOP: now also J10-4.S, J6-2.S, J7-2.S; no longer X10A-G$2.S, X11A-G$2.S, X13A-G$2.S

Commit message: rev.003 RC1
Parts:
- removed X6A-: REKOJESC_LEW, my_electronics_library:43045-0812
- added D3, D4: 1N4446, diode:1N4446
Connections:
- new net N$2: D3.C, J10-4.S
- new net N$3: D4.C, J10-2.S
- net +12V/ST: now also J1-3.S, J13-1.S, J13-2.S, J13-3.S; no longer J1-1.S, X6A-G$1.S, X6A-G$4.S
- net KIER_LEWY: now also J13-7.S; no longer X6A-G$7.S
- net KIER_PRAWY: now also J13-8.S; no longer X6A-G$5.S
- net KIER_WSPOLNY: now also J1-1.S, J13-4.S; no longer J1-3.S, X6A-G$6.S
- net KLAKSON: now also J13-5.S; no longer X6A-G$3.S
- net MIJANIA: now also D4.A, J13-6.S; no longer J10-2.S, X6A-G$2.S
- net STOP: now also D3.A; no longer J10-4.S
Other:
- moved on the sheet: J1-1, J1-2, J1-3, J13-1, J13-2, J13-3, J13-4, J13-5, J13-6, J13-7, J13-8

Commit message: rev.003 RC2
Connections:
- net N$2 renamed STOP_DIODE
- net N$3 renamed MIJANIA_DIODE
Changed lines of the file:
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@@
 <label x="264.16" y="147.32" size="2.54" layer="95" rot="R90"/>
 <label x="467.36" y="177.8" size="2.54" layer="95"/>
-<label x="469.9" y="93.98" size="2.54" layer="95"/>
+<label x="449.58" y="93.98" size="2.54" layer="95"/>
 <wire x1="269.24" y1="182.88" x2="269.24" y2="205.74" width="0.1524" layer="91"/>
 <pinref part="J11" gate="-5" pin="S"/>
@@
 <label x="320.04" y="134.62" size="2.54" layer="95" rot="R90"/>
 <label x="347.98" y="134.62" size="2.54" layer="95" rot="R90"/>
-<label x="472.44" y="78.74" size="2.54" layer="95"/>
+<label x="441.96" y="78.74" size="2.54" layer="95"/>
 <pinref part="J6" gate="-2" pin="S"/>
 <pinref part="J7" gate="-2" pin="S"/>
@@
 </segment>
 </net>
-<net name="N$2" class="0">
+<net name="STOP_DIODE" class="0">
 <segment>
 <pinref part="D3" gate="1" pin="C"/>
 <pinref part="J10" gate="-4" pin="S"/>
 <wire x1="457.2" y1="78.74" x2="482.6" y2="78.74" width="0.1524" layer="91"/>
+<label x="467.36" y="78.74" size="1.778" layer="95"/>
 </segment>
 </net>
-<net name="N$3" class="0">
+<net name="MIJANIA_DIODE" class="0">
 <segment>
 <pinref part="D4" gate="1" pin="C"/>
 <pinref part="J10" gate="-2" pin="S"/>
 <wire x1="467.36" y1="93.98" x2="482.6" y2="93.98" width="0.1524" layer="91"/>
+<label x="472.44" y="93.98" size="1.778" layer="95"/>
 </segment>
 </net>

Commit message: poprawki diod, ver.003 RC3
Parts:
- D1, D4: value 1N4446 -> 1N4004; device diode:1N4446 -> diode:1N4004
- D2, D3: value 1N4446 -> BYV28-200; device diode:1N4446 -> diode:BYV28
Connections:
- net KIER_LEWY: now also D4.A; no longer D1.A
- net KIER_PRAWY: now also D1.A; no longer D2.A
- net MIJANIA: now also D3.A; no longer D4.A
- net MIJANIA_DIODE: now also D3.C; no longer D4.C
- net N$1: now also D4.C; no longer D2.C
- net STOP: now also D2.A; no longer D3.A
- net STOP_DIODE: now also D2.C; no longer D3.C
Other:
- moved on the sheet: D1, D2, D3, D4
Changed lines of the file:
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@@
 <parts>
 <part name="X1B" library="con-molex" deviceset="5566-2" device=""/>
-<part name="D1" library="diode" deviceset="1N4446" device=""/>
-<part name="D2" library="diode" deviceset="1N4446" device=""/>
 <part name="J1" library="con-molex" library_urn="urn:adsk.eagle:library:165" deviceset="22-?-03" device="27-2031" value="PRZERYWACZ"/>
 <part name="J2" library="con-molex" library_urn="urn:adsk.eagle:library:165" deviceset="22-?-02" device="27-2021" value="STACYJKA"/>
@@
 <part name="J12" library="con-molex" library_urn="urn:adsk.eagle:library:165" deviceset="22-?-06" device="27-2061" value="SYGNALIZATOR"/>
 <part name="J13" library="con-molex" library_urn="urn:adsk.eagle:library:165" deviceset="22-?-08" device="27-2081"/>
-<part name="D3" library="diode" deviceset="1N4446" device=""/>
-<part name="D4" library="diode" deviceset="1N4446" device=""/>
+<part name="D4" library="diode" library_urn="urn:adsk.eagle:library:210" deviceset="1N4004" device="" package3d_urn="urn:adsk.eagle:package:43336/1"/>
+<part name="D1" library="diode" library_urn="urn:adsk.eagle:library:210" deviceset="1N4004" device="" package3d_urn="urn:adsk.eagle:package:43336/1"/>
+<part name="D2" library="diode" library_urn="urn:adsk.eagle:library:210" deviceset="BYV28" device="" package3d_urn="urn:adsk.eagle:package:43385/1" value="BYV28-200"/>
+<part name="D3" library="diode" library_urn="urn:adsk.eagle:library:210" deviceset="BYV28" device="" package3d_urn="urn:adsk.eagle:package:43385/1" value="BYV28-200"/>
 </parts>
 <sheets>
@@
 <instance part="X1B" gate="-1" x="-35.56" y="93.98" rot="R180"/>
 <instance part="X1B" gate="-2" x="-35.56" y="88.9" rot="R180"/>
-<instance part="D1" gate="1" x="365.76" y="116.84" rot="R90"/>
-<instance part="D2" gate="1" x="370.84" y="116.84" rot="R90"/>
 <instance part="J1" gate="-1" x="48.26" y="137.16" rot="R90"/>
 <instance part="J1" gate="-2" x="40.64" y="137.16" rot="R90"/>
@@
 <instance part="J13" gate="-7" x="175.26" y="213.36" rot="R90"/>
 <instance part="J13" gate="-8" x="165.1" y="213.36" rot="R90"/>
-<instance part="D3" gate="1" x="454.66" y="78.74"/>
-<instance part="D4" gate="1" x="464.82" y="93.98"/>
+<instance part="D4" gate="1" x="365.76" y="116.84" rot="R90"/>
+<instance part="D1" gate="1" x="370.84" y="116.84" rot="R90"/>
+<instance part="D2" gate="1" x="454.66" y="78.74"/>
+<instance part="D3" gate="1" x="464.82" y="93.98"/>
 </instances>
 <busses>
@@
 <pinref part="J12" gate="-6" pin="S"/>
 <pinref part="J13" gate="-6" pin="S"/>
-<pinref part="D4" gate="1" pin="A"/>
 <wire x1="462.28" y1="93.98" x2="452.12" y2="93.98" width="0.1524" layer="91"/>
 <junction x="452.12" y="93.98"/>
+<pinref part="D3" gate="1" pin="A"/>
 </segment>
 </net>
@@
 <wire x1="274.32" y1="180.34" x2="274.32" y2="205.74" width="0.1524" layer="91"/>
 <label x="350.52" y="109.22" size="1.778" layer="95"/>
-<pinref part="D1" gate="1" pin="A"/>
 <wire x1="365.76" y1="114.3" x2="365.76" y2="109.22" width="0.1524" layer="91"/>
 <junction x="365.76" y="109.22"/>
@@
 <pinref part="J12" gate="-1" pin="S"/>
 <pinref part="J13" gate="-7" pin="S"/>
+<pinref part="D4" gate="1" pin="A"/>
 </segment>
 </net>
@@
 <wire x1="279.4" y1="177.8" x2="279.4" y2="205.74" width="0.1524" layer="91"/>
 <label x="350.52" y="104.14" size="1.778" layer="95"/>
-<pinref part="D2" gate="1" pin="A"/>
 <wire x1="370.84" y1="114.3" x2="370.84" y2="104.14" width="0.1524" layer="91"/>
 <junction x="370.84" y="104.14"/>
@@
 <pinref part="J12" gate="-2" pin="S"/>
 <pinref part="J13" gate="-8" pin="S"/>
+<pinref part="D1" gate="1" pin="A"/>
 </segment>
 </net>
@@
 <pinref part="J6" gate="-2" pin="S"/>
 <pinref part="J7" gate="-2" pin="S"/>
-<pinref part="D3" gate="1" pin="A"/>
 <wire x1="452.12" y1="78.74" x2="436.88" y2="78.74" width="0.1524" layer="91"/>
+<pinref part="D2" gate="1" pin="A"/>
 </segment>
 </net>
 <net name="N$1" class="0">
 <segment>
-<pinref part="D1" gate="1" pin="C"/>
-<pinref part="D2" gate="1" pin="C"/>
 <wire x1="365.76" y1="119.38" x2="370.84" y2="119.38" width="0.1524" layer="91"/>
 <wire x1="370.84" y1="119.38" x2="378.46" y2="119.38" width="0.1524" layer="91"/>
 <wire x1="378.46" y1="119.38" x2="378.46" y2="157.48" width="0.1524" layer="91"/>
+<pinref part="J4" gate="-2" pin="S"/>
+<pinref part="D4" gate="1" pin="C"/>
+<pinref part="D1" gate="1" pin="C"/>
 <junction x="370.84" y="119.38"/>
-<pinref part="J4" gate="-2" pin="S"/>
 </segment>
 </net>
 <net name="STOP_DIODE" class="0">
 <segment>
-<pinref part="D3" gate="1" pin="C"/>
 <pinref part="J10" gate="-4" pin="S"/>
 <wire x1="457.2" y1="78.74" x2="482.6" y2="78.74" width="0.1524" layer="91"/>
 <label x="467.36" y="78.74" size="1.778" layer="95"/>
+<pinref part="D2" gate="1" pin="C"/>
 </segment>
 </net>
 <net name="MIJANIA_DIODE" class="0">
 <segment>
-<pinref part="D4" gate="1" pin="C"/>
 <pinref part="J10" gate="-2" pin="S"/>
 <wire x1="467.36" y1="93.98" x2="482.6" y2="93.98" width="0.1524" layer="91"/>
 <label x="472.44" y="93.98" size="1.778" layer="95"/>
+<pinref part="D3" gate="1" pin="C"/>
 </segment>
 </net>
@@
 with this version.
 </note>
+<note version="8.3" severity="warning">
+Since Version 8.3, EAGLE supports URNs for individual library
+assets (packages, symbols, and devices). The URNs of those assets
+will not be understood (or retained) with this version.
+</note>
+<note version="8.3" severity="warning">
+Since Version 8.3, EAGLE supports the association of 3D packages
+with devices in libraries, schematics, and board files. Those 3D
+packages will not be understood (or retained) with this version.
+</note>
 </compatibility>
